File: COGDisplayBreakout.kicad_pcb (KiCad board)
At the start: 2 copper layers, 29.2 x 31.8 mm, 17 parts, among them J1 SPI_Header, U1 APX803S

Commit message: Adds a SN field and label text, v1.2
Other:
- board text added: "COG Display Breakout V.1.2"
- board text added: "S/N"
Changed lines of the file:
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@@
 		)
+	)
+	(gr_rect
+		(start 134.62 97.79)
+		(end 143.002 100.33)
+		(stroke
+			(width 0.1)
+			(type solid)
+		)
+		(fill yes)
+		(layer "B.SilkS")
 	)
 	(gr_arc
@@
 	)
 	(gr_text "12"
-		(at 144.78 90.424 0)
-		(layer "B.SilkS")
-		(effects
-			(font
-				(size 0.8 0.8)
+		(at 146.05 90.678 0)
+		(layer "B.SilkS")
+		(effects
+			(font
+				(size 0.8 0.8)
+				(thickness 0.1)
+			)
+			(justify left bottom mirror)
+		)
+	)
+	(gr_text "COG Display\nBreakout\nV.1.2"
+		(at 146.558 88.646 0)
+		(layer "B.SilkS")
+		(effects
+			(font
+				(size 1 1)
 				(thickness 0.1)
 			)
@@
 		)
 	)
+	(gr_text "S/N"
+		(at 143.002 97.028 0)
+		(layer "B.SilkS")
+		(effects
+			(font
+				(size 1 1)
+				(thickness 0.1)
+			)
+			(justify left bottom mirror)
+		)
+	)
 	(gr_text "1"
-		(at 152.4 90.424 0)
-		(layer "B.SilkS")
-		(effects
+		(at 152.146 90.678 0)
+		(layer "B.SilkS")
+		(effects
